File: LT8705.kicad_pcb (KiCad board)
At the start: 4 copper layers, 64 parts, among them J1 XH-2, J2 HDR-M-2.54-1*4P, Q1 CSD19532Q5B, Q2 CSD19532Q5B, Q3 CSD19532Q5B, Q4 CSD19532Q5B, U1 LT8705EFE

Commit message: 1
Parts:
- moved C32 153.7 mm to (118.9, 107.4), turned to 180 degrees
- moved R15 153.5 mm to (118.9, 109.0), turned to 180 degrees
- moved R16 133.6 mm to (122.4, 109.7), turned to 180 degrees
- moved D1 124.1 mm to (110.8, 102.0), turned to 270 degrees
- moved R14 122.9 mm to (118.9, 98.0)
- moved D2 121.5 mm to (113.4, 102.0), turned to 270 degrees
- moved R10 121.0 mm to (118.9, 101.1), turned to 180 degrees
- moved R9 118.8 mm to (118.9, 99.6)
- moved R13 114.3 mm to (122.4, 111.3), turned to 180 degrees
- moved R17 104.8 mm to (171.3, 105.6), turned to 180 degrees
- moved R8 104.3 mm to (118.9, 104.4), turned to 180 degrees
- moved C29 104.3 mm to (118.9, 105.9), turned to 180 degrees
- moved C31 104.2 mm to (170.0, 113.6), turned to 270 degrees
- moved RV2 103.6 mm to (175.1, 109.2)
- moved C33 102.6 mm to (172.5, 113.6), turned to 270 degrees
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
Commit message: 1
Parts:
- removed the C8 at (106.4, 77.5)
- removed the R6 at (137.2, 84.3)
- removed the R7 at (149.6, 68.3)
- added C10: 4.7uF/100V, Capacitor_SMD:C_1210_3225Metric_Pad1.33x2.70mm_HandSolder, B.Cu at (116.6, 59.8)
- added C5: 4.7uF/100V, Capacitor_SMD:C_1210_3225Metric_Pad1.33x2.70mm_HandSolder, F.Cu at (107.6, 72.3)
- added C9: 4.7uF/100V, Capacitor_SMD:C_1210_3225Metric_Pad1.33x2.70mm_HandSolder, B.Cu at (116.6, 63.1)
- added D1: ?, Diode_SMD:D_SMA-SMB_Universal_Handsoldering, F.Cu at (115.1, 76.9)
- added D2: ?, Diode_SMD:D_SMA-SMB_Universal_Handsoldering, F.Cu at (142.6, 76.5)
- added Q3: NC, Package_TO_SOT_SMD:TDSON-8-1, B.Cu at (123.3, 67.3)
- added Q5: NC, Package_TO_SOT_SMD:TDSON-8-1, B.Cu at (134.6, 69.2)
- added Q6: NC, Package_TO_SOT_SMD:TDSON-8-1, F.Cu at (137.4, 78.2)
- added Q8: CSD19532Q5B, Package_TO_SOT_SMD:TDSON-8-1, F.Cu at (131.7, 78.2)
- added R10: 2R, Resistor_SMD:R_0603_1608Metric_Pad0.98x0.95mm_HandSolder, F.Cu at (123.2, 108.0)
- added R11: 0, Resistor_SMD:R_0603_1608Metric_Pad0.98x0.95mm_HandSolder, B.Cu at (135.6, 58.2)
- added R12: 2R, Resistor_SMD:R_0603_1608Metric_Pad0.98x0.95mm_HandSolder, F.Cu at (124.7, 108.0)
- added R13: WSK06125L000FEA, Resistor_SMD:R_Shunt_Vishay_WSKW0612, F.Cu at (141.4, 64.8)
- added R3: 0, Resistor_SMD:R_0603_1608Metric_Pad0.98x0.95mm_HandSolder, F.Cu at (120.1, 107.9)
- added R4: 2R, Resistor_SMD:R_0603_1608Metric_Pad0.98x0.95mm_HandSolder, B.Cu at (122.3, 71.0)
- added R8: WSK06125L000FEA, Resistor_SMD:R_Shunt_Vishay_WSKW0612, F.Cu at (128.9, 85.1)
- added R9: 0, Resistor_SMD:R_0603_1608Metric_Pad0.98x0.95mm_HandSolder, B.Cu at (135.6, 65.5)
- added RV1: 50K, Potentiometer_THT:Potentiometer_Bourns_3296W_Vertical, F.Cu at (105.7, 111.8)
- C18: renamed from C16; value C -> 100nF
- C26: renamed from C24; moved to B.Cu
- C27: renamed from C25; moved to B.Cu
- C28: renamed from C26; moved to B.Cu
- C29: renamed from C27; moved to B.Cu
- C3, C4, C6: footprint Capacitor_SMD:C_1210_3225Metric_Pad1.42x2.65mm_HandSolder -> Capacitor_SMD:C_1210_3225Metric_Pad1.33x2.70mm_HandSolder
- C7: renamed from C10; footprint Capacitor_SMD:C_1210_3225Metric_Pad1.42x2.65mm_HandSolder -> Capacitor_SMD:C_1210_3225Metric_Pad1.33x2.70mm_HandSolder; moved to B.Cu
- C8: renamed from C12; footprint Capacitor_SMD:C_1210_3225Metric_Pad1.42x2.65mm_HandSolder -> Capacitor_SMD:C_1210_3225Metric_Pad1.33x2.70mm_HandSolder; moved to B.Cu
- Q1: moved to B.Cu
- Q4: value CSD19532Q5B -> NC
- Q7: renamed from Q3; moved to B.Cu
- R1: value WSK06121L000FEA -> WSK06125L000FEA; footprint _Acha:WSK06121L000FEA -> Resistor_SMD:R_Shunt_Vishay_WSKW0612
- R14: renamed from R8; footprint Resistor_SMD:R_0603_1608Metric_Pad1.05x0.95mm_HandSolder -> Resistor_SMD:R_0603_1608Metric_Pad0.98x0.95mm_HandSolder
- R15: renamed from R9; footprint Resistor_SMD:R_0603_1608Metric_Pad1.05x0.95mm_HandSolder -> Resistor_SMD:R_0603_1608Metric_Pad0.98x0.95mm_HandSolder
- R16: renamed from R10; footprint Resistor_SMD:R_0603_1608Metric_Pad1.05x0.95mm_HandSolder -> Resistor_SMD:R_0603_1608Metric_Pad0.98x0.95mm_HandSolder
- R17: renamed from R11; footprint Resistor_SMD:R_0603_1608Metric_Pad1.05x0.95mm_HandSolder -> Resistor_SMD:R_0603_1608Metric_Pad0.98x0.95mm_HandSolder
- R18: renamed from R12; footprint Resistor_SMD:R_0603_1608Metric_Pad1.05x0.95mm_HandSolder -> Resistor_SMD:R_0603_1608Metric_Pad0.98x0.95mm_HandSolder
- R19: renamed from R13; footprint Resistor_SMD:R_0603_1608Metric_Pad1.05x0.95mm_HandSolder -> Resistor_SMD:R_0603_1608Metric_Pad0.98x0.95mm_HandSolder
- R2: footprint Resistor_SMD:R_0603_1608Metric_Pad1.05x0.95mm_HandSolder -> Resistor_SMD:R_0603_1608Metric_Pad0.98x0.95mm_HandSolder; moved to B.Cu
- R20: renamed from R14; footprint Resistor_SMD:R_0603_1608Metric_Pad1.05x0.95mm_HandSolder -> Resistor_SMD:R_0603_1608Metric_Pad0.98x0.95mm_HandSolder
- R21: renamed from R15; value 40.2K -> NC; footprint Resistor_SMD:R_0603_1608Metric_Pad1.05x0.95mm_HandSolder -> Resistor_SMD:R_0603_1608Metric_Pad0.98x0.95mm_HandSolder
- R22: renamed from R16; footprint Resistor_SMD:R_0603_1608Metric_Pad1.05x0.95mm_HandSolder -> Resistor_SMD:R_0603_1608Metric_Pad0.98x0.95mm_HandSolder
- R23: renamed from R17; footprint Resistor_SMD:R_0603_1608Metric_Pad1.05x0.95mm_HandSolder -> Resistor_SMD:R_0603_1608Metric_Pad0.98x0.95mm_HandSolder
- R24: renamed from R18; footprint Resistor_SMD:R_0603_1608Metric_Pad1.05x0.95mm_HandSolder -> Resistor_SMD:R_0603_1608Metric_Pad0.98x0.95mm_HandSolder
- R25: renamed from R19; footprint Resistor_SMD:R_0603_1608Metric_Pad1.05x0.95mm_HandSolder -> Resistor_SMD:R_0603_1608Metric_Pad0.98x0.95mm_HandSolder
- R5: value WSK06121L000FEA -> 0; footprint _Acha:WSK06121L000FEA -> Resistor_SMD:R_0603_1608Metric_Pad0.98x0.95mm_HandSolder
- R6: renamed from R3; footprint Resistor_SMD:R_0603_1608Metric_Pad1.05x0.95mm_HandSolder -> Resistor_SMD:R_0603_1608Metric_Pad0.98x0.95mm_HandSolder
- R7: renamed from R4; footprint Resistor_SMD:R_0603_1608Metric_Pad1.05x0.95mm_HandSolder -> Resistor_SMD:R_0603_1608Metric_Pad0.98x0.95mm_HandSolder
- moved C17 128.4 mm to (38.4, 57.5), turned to 90 degrees
- moved C1 61.7 mm to (38.5, 76.1)
- moved D3 34.5 mm to (145.3, 103.0), turned to 90 degrees
- moved D4 29.5 mm to (142.9, 103.0), turned to 90 degrees
- moved J2 23.6 mm to (93.0, 102.7)
- moved R5 21.5 mm to (121.7, 108.0), turned to 90 degrees
- moved C2 21.4 mm to (108.2, 65.3), turned to 90 degrees
- moved C29 17.9 mm to (141.4, 59.8), turned to 0 degrees
- moved C28 15.8 mm to (141.4, 63.1), turned to 0 degrees
- moved C26 15.6 mm to (141.4, 69.7), turned to 0 degrees
- moved R23 15.0 mm to (156.3, 105.0)
- moved C27 15.0 mm to (141.4, 66.4), turned to 0 degrees
- moved J1 15.0 mm to (139.3, 120.1)
- moved RV3 15.0 mm to (160.1, 109.2)
- moved C33 14.8 mm to (155.2, 113.2), turned to 180 degrees
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- renumbered C5 to C11, C7 to C12, C9 to C13, C11 to C14, C13 to C15, C14 to C16, C15 to C17, C17 to C19, C18 to C20, C19 to C21, C20 to C22, C21 to C23, C22 to C24, C23 to C25, C28 to C30, C29 to C31, C30 to C32, C31 to C33, C33 to C34, C32 to C35, D1 to D3, D2 to D4, RV1 to RV2, RV2 to RV3
Connections:
- Q2 pad 1: Net-(Q2-Pad1) -> Net-(D1-Pad2)
- Q2 pad 2: Net-(Q2-Pad1) -> Net-(D1-Pad2)
- Q2 pad 3: Net-(Q2-Pad1) -> Net-(D1-Pad2)
- Q2 pad 4: /BG1 -> Net-(Q2-Pad4)
- Q4 pad 1: Net-(Q2-Pad1) -> Net-(D1-Pad2)
- Q4 pad 2: Net-(Q2-Pad1) -> Net-(D1-Pad2)
- Q4 pad 3: Net-(Q2-Pad1) -> Net-(D1-Pad2)
- Q4 pad 5: /SW2 -> /SW1
- Q7 pad 4: /TG2 -> Net-(Q7-Pad4)
- R6 pad 1: Net-(R3-Pad1) -> Net-(R6-Pad1)
- R7 pad 1: Net-(R4-Pad1) -> Net-(R7-Pad1)
Routing:
- net Net-(Q4-Pad4): track 1.80 -> 0.00 mm
- net Net-(Q1-Pad4): track 1.70 -> 0.00 mm
- removed copper zone on F.Cu, net /SW1
- removed copper zone on F.Cu, net /SW2
- removed copper zone on F.Cu, net Net-(Q2-Pad1)

Commit message: Updated
Parts:
- removed C1, C17: 220uF/100V, Capacitor_THT:C_Radial_D12.5mm_H25.0mm_P5.00mm
- moved C35 53.1 mm to (163.6, 112.5)
- moved R21 53.1 mm to (163.6, 111.0)
- moved RV1 53.1 mm to (158.8, 110.7)
- moved R23 33.7 mm to (123.9, 114.2)
- moved RV3 33.7 mm to (127.7, 118.3)
- moved C33 33.7 mm to (122.8, 122.3)
- moved C34 33.7 mm to (126.2, 122.3)
- moved R4 23.7 mm to (130.6, 48.8)
- moved R9 18.1 mm to (142.9, 49.0)
- moved C30 18.0 mm to (106.4, 88.4)
- moved R17 18.0 mm to (106.4, 89.9)
- moved R18 18.0 mm to (106.4, 91.4)
- moved R2 14.4 mm to (124.7, 49.4)
- moved R11 10.4 mm to (137.1, 47.9)
- moved C31 4.34 mm to (106.3, 101.5)
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Connections:
- C10 pad 1: VDD -> Net-(C10-Pad1)
- C7 pad 1: VDD -> Net-(C10-Pad1)
- C8 pad 1: VDD -> Net-(C10-Pad1)
- C9 pad 1: VDD -> Net-(C10-Pad1)
- Q1 pad 5: Net-(Q1-Pad5) -> Net-(C10-Pad1)
- Q3 pad 5: Net-(Q1-Pad5) -> Net-(C10-Pad1)
- R1 pad 4: Net-(Q1-Pad5) -> Net-(C10-Pad1)
Routing:
- net VDD: vias 0 -> 16
- added copper zone on B.Cu, net Net-(C10-Pad1)
- added copper zone on F.Cu, net Net-(C10-Pad1)
- added copper zone on B.Cu, net VDD
- added copper zone on F.Cu, net VDD

Commit message: updated
Parts:
- removed the C21 at (150.0, 65.3)
- added C25: 220uF/100V, Capacitor_THT:C_Radial_D12.5mm_H25.0mm_P5.00mm, F.Cu at (150.0, 65.3)
- added R26: 0, Resistor_SMD:R_0603_1608Metric_Pad0.98x0.95mm_HandSolder, F.Cu at (105.8, 118.1)
- C17: renamed from C22; moved to B.Cu
- C18: renamed from C23; moved to B.Cu
- C19: renamed from C24; moved to B.Cu
- C20: renamed from C25; moved to B.Cu
- C26, C27, C28, C29, R11, R2, R4, R9: moved to F.Cu
- R1: value WSK06125L000FEA -> 0R; footprint Resistor_SMD:R_Shunt_Vishay_WSKW0612 -> _Acha:R_0612_1632Metric
- R13: value WSK06125L000FEA -> R005; footprint Resistor_SMD:R_Shunt_Vishay_WSKW0612 -> _Acha:R_0612_1632Metric
- R8: value WSK06125L000FEA -> R005; footprint Resistor_SMD:R_Shunt_Vishay_WSKW0612 -> _Acha:R_1225_3263Metric
- moved R11 53.7 mm to (136.8, 101.6), turned to 0 degrees
- moved R9 51.3 mm to (136.8, 99.9), turned to 0 degrees
- moved R4 49.9 mm to (136.8, 98.3)
- moved R2 48.8 mm to (136.8, 96.6)
- moved C16 18.3 mm to (119.0, 92.3), turned to 180 degrees
- moved C15 18.0 mm to (119.0, 96.9), turned to 180 degrees
- moved R7 17.7 mm to (119.0, 93.9), turned to 0 degrees
- moved R6 17.5 mm to (119.0, 95.4), turned to 0 degrees
- moved C26 15.6 mm to (156.7, 72.4), turned to 270 degrees
- moved C17 15.2 mm to (141.7, 69.8), turned to 0 degrees
- moved C29 13.7 mm to (146.8, 72.4), turned to 270 degrees
- moved C27 13.5 mm to (153.4, 72.4), turned to 270 degrees
- moved C20 13.3 mm to (141.7, 59.9), turned to 0 degrees
- moved C18 13.0 mm to (141.7, 66.5), turned to 0 degrees
- moved C28 12.8 mm to (150.1, 72.4), turned to 270 degrees
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- renumbered C9 to C10, C12 to C11, C10 to C12, C18 to C21, C19 to C22, C20 to C23, C11 to C9
Connections:
- C10 pad 1: Net-(C10-Pad1) -> /CSNIN
- C10 pad 2: GNDA -> GNDPWR
- C12 pad 1: Net-(C10-Pad1) -> /CSNIN
- C12 pad 2: GNDA -> GNDPWR
- C17 pad 1: VD -> /CSPOUT
- C17 pad 2: GNDA -> GNDPWR
- C18 pad 1: VD -> /CSPOUT
- C18 pad 2: GNDA -> GNDPWR
- C19 pad 1: VD -> /CSPOUT
- C19 pad 2: GNDA -> GNDPWR
- C2 pad 2: GNDA -> GNDPWR
- C20 pad 1: VD -> /CSPOUT
- C20 pad 2: GNDA -> GNDPWR
- C26 pad 2: GNDA -> GNDPWR
- C27 pad 2: GNDA -> GNDPWR
- C28 pad 2: GNDA -> GNDPWR
- C29 pad 2: GNDA -> GNDPWR
- C3 pad 2: GNDA -> GNDPWR
- C4 pad 2: GNDA -> GNDPWR
- C5 pad 2: GNDA -> GNDPWR
- C6 pad 2: GNDA -> GNDPWR
- C7 pad 1: Net-(C10-Pad1) -> /CSNIN
- C7 pad 2: GNDA -> GNDPWR
- C8 pad 1: Net-(C10-Pad1) -> /CSNIN
- C8 pad 2: GNDA -> GNDPWR
- D2 pad 2: Net-(D2-Pad2) -> /CSPOUT
- Q1 pad 5: Net-(C10-Pad1) -> /CSNIN
- Q3 pad 5: Net-(C10-Pad1) -> /CSNIN
- Q5 pad 5: Net-(D2-Pad2) -> /CSPOUT
- Q7 pad 5: Net-(D2-Pad2) -> /CSPOUT
- R1 pad 1: VDD -> /CSNIN
- R1 pad 2: /CSPIN -> VDD
- R13 pad 1: Net-(D2-Pad2) -> VD
- R6 pad 1: Net-(R6-Pad1) -> Net-(D1-Pad2)
- R7 pad 1: Net-(R7-Pad1) -> GNDPWR
- R8 pad 1: GNDA -> GNDPWR
- R8 pad 2: Net-(R7-Pad1) -> Net-(D1-Pad2)
- U1 pad 32: /CSNOUT -> VD
- U1 pad 37: /CSPIN -> VDD
Routing:
- net Net-(Q6-Pad4): track 0.00 -> 38.4 mm, vias 0 -> 2
- net Net-(Q8-Pad4): track 0.00 -> 34.0 mm, vias 0 -> 2
- net Net-(Q2-Pad4): track 0.00 -> 32.0 mm, vias 0 -> 2
- net /BOOST1: track 0.00 -> 28.2 mm, vias 0 -> 2
- net Net-(Q4-Pad4): track 0.00 -> 28.1 mm, vias 0 -> 2
- net /BOOST2: track 0.00 -> 22.2 mm
- net /BG1: track 0.00 -> 11.1 mm
- net /GATEVCC: track 0.00 -> 9.80 mm
- net /CSN: track 0.00 -> 9.00 mm
- net /CSP: track 0.00 -> 9.00 mm
- net /TG1: track 0.00 -> 5.13 mm
- net /TG2: track 0.00 -> 5.03 mm
- net /EXTVCC: track 0.00 -> 4.58 mm
- net /BG2: track 0.00 -> 4.48 mm
- net /RT: track 0.00 -> 3.47 mm
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- added copper zone on B.Cu, net /CSNIN
- added copper zone on F.Cu, net /CSNIN
- added copper zone on B.Cu, net /CSPOUT
- added copper zone on F.Cu, net /CSPOUT
- added copper zone on B.Cu, net /SW1
- added copper zone on F.Cu, net /SW1
- added copper zone on B.Cu, net /SW2
- added copper zone on F.Cu, net /SW2
- added copper zone on F.Cu, net Net-(D1-Pad2)
- removed copper zone on B.Cu, net Net-(C10-Pad1)
- removed copper zone on F.Cu, net Net-(C10-Pad1)

Commit message: 1
Parts:
- moved R24 40.1 mm to (161.3, 80.1), turned to 270 degrees
- moved RV2 39.7 mm to (165.1, 80.8), turned to 90 degrees
- moved R25 38.2 mm to (161.3, 83.6), turned to 270 degrees
- moved RV1 20.1 mm to (165.1, 91.7), turned to 90 degrees
- moved R21 20.1 mm to (161.3, 91.1), turned to 90 degrees
- moved J1 19.0 mm to (153.3, 107.2), turned to 90 degrees
- moved C35 18.2 mm to (161.3, 94.5), turned to 270 degrees
- moved J2 17.4 mm to (105.4, 90.6)
- moved R23 17.0 mm to (138.1, 104.8)
- moved RV3 17.0 mm to (141.9, 108.9)
- moved C33 17.0 mm to (137.0, 112.9)
- moved C34 17.0 mm to (140.5, 112.9)
- moved R15 7.18 mm to (113.4, 93.9)
- moved C31 7.17 mm to (113.4, 100.6)
- moved R14 7.17 mm to (113.4, 99.1)
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Routing:
- net VDD: track 1.52 -> 78.2 mm, vias 17 -> 20
- net /SW2: track 2.99 -> 54.4 mm, vias 48 -> 49
- net /CSNIN: track 0.00 -> 49.4 mm, vias 17 -> 18
- net Net-(Q7-Pad4): track 1.35 -> 50.1 mm
- net /SW1: track 2.26 -> 47.1 mm, vias 48 -> 49
- net VD: track 0.00 -> 44.4 mm, vias 1 -> 2
- net Net-(Q1-Pad4): track 1.45 -> 42.5 mm
- net Net-(Q5-Pad4): track 1.41 -> 41.9 mm
- net Net-(D3-Pad2): track 0.87 -> 40.8 mm, vias 1 -> 2
- net /CSPOUT: track 0.00 -> 39.5 mm, vias 17 -> 18
- net Net-(Q3-Pad4): track 1.38 -> 39.0 mm
- net /VC: track 0.00 -> 33.2 mm, vias 0 -> 2
- net /MODE: track 0.00 -> 26.5 mm, vias 0 -> 1
- net Net-(D1-Pad2): track 0.00 -> 23.5 mm, vias 1 -> 2
- net /LDO33: track 3.42 -> 24.3 mm, vias 0 -> 2
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
Commit message: 1
Parts:
- removed the R26 at (106.3, 111.5)
- added R22: R, Resistor_SMD:R_0603_1608Metric_Pad0.98x0.95mm_HandSolder, F.Cu at (160.4, 93.1)
- moved J1 16.5 mm to (164.1, 94.7)
- moved C35 9.78 mm to (161.3, 104.3)
- moved R23 9.78 mm to (161.3, 100.8)
- moved RV1 9.78 mm to (165.1, 101.5)
- renumbered R9 to R10, R10 to R11, R11 to R12, R12 to R13, R13 to R14, R14 to R15, R15 to R16, R16 to R17, R17 to R18, R18 to R19, R1 to R2, R19 to R20, R20 to R21, R21 to R23, R22 to R24, R23 to R25, R24 to R26, R25 to R27, R2 to R3, R3 to R4, R4 to R5, R5 to R6, R6 to R7, R7 to R8, R8 to R9
Routing:
- net /FBOUT: track 8.31 -> 56.2 mm, vias 1 -> 2
- net /IMON_OUT: track 8.97 -> 51.4 mm, vias 1 -> 2
- net /EXTVCC: track 4.58 -> 43.6 mm, vias 0 -> 1
- net VD: track 44.4 -> 60.7 mm
- net Net-(C34-Pad1): track 4.09 -> 8.37 mm

Commit message: 1
Parts:
- added C1: 220uF/100V, Capacitor_THT:C_Radial_D12.5mm_H25.0mm_P5.00mm, F.Cu at (105.5, 80.5)
- added C24: 220uF/100V, Capacitor_THT:C_Radial_D12.5mm_H25.0mm_P5.00mm, F.Cu at (152.0, 80.6)
- moved R26 14.9 mm to (154.0, 93.1)
- moved R27 14.9 mm to (154.0, 96.5)
- moved RV2 14.9 mm to (157.8, 93.7)
- moved R22 14.0 mm to (161.7, 107.1)
- moved J1 14.0 mm to (165.4, 108.7)
- moved C35 7.88 mm to (162.8, 96.5)
- moved R23 7.88 mm to (162.8, 93.1)
- moved RV1 7.88 mm to (166.6, 93.7)
- moved J2 4.78 mm to (105.9, 95.3)
- moved C2 2.74 mm to (105.5, 65.1)
- moved C25 1.92 mm to (151.9, 65.1)
- moved C30 0.76 mm to (113.4, 89.0)
- moved R18 0.76 mm to (113.4, 90.6)
- moved R19 0.76 mm to (113.4, 92.1)
Routing:
- net /CSPOUT: track 39.5 -> 0.00 mm, vias 18 -> 17
- net VDD: track 78.2 -> 49.9 mm, vias 20 -> 2
- net /MODE: track 26.5 -> 4.34 mm
- net VD: track 60.7 -> 39.3 mm
- net /IMON_OUT: track 51.4 -> 65.7 mm, vias 2 -> 1
- net /SHDN: track 15.5 -> 3.52 mm, vias 2 -> 0
- net /EXTVCC: track 43.6 -> 55.5 mm, vias 1 -> 2
- net /LDO33: track 24.3 -> 29.6 mm
- net /FBOUT: track 56.2 -> 53.6 mm, vias 2 -> 1
- net GNDPWR: track 20.6 -> 23.1 mm
- net Net-(Q3-Pad4): track 39.0 -> 36.9 mm
- net Net-(D1-Pad2): track 23.5 -> 25.3 mm
- net Net-(Q1-Pad4): track 42.5 -> 41.0 mm
- net /SW2: track 54.4 -> 55.4 mm
- added copper zone on B.Cu, net GNDPWR
- added copper zone on F.Cu, net GNDPWR
- added copper zone on F.Cu, net VD
- removed copper zone on B.Cu, net VDD
Other:
- net class Default: trace_width 0.25 -> 0.2; via_dia 0.8 -> 0.6; via_drill 0.4 -> 0.3
- net class POWER added: clearance 0.25, trace_width 0.2, via_dia 0.6, via_drill 0.3
- net class POWER2 added: clearance 0.2, trace_width 0.35, via_dia 0.6, via_drill 0.3

Commit message: 1
Parts:
- moved R2 5.01 mm to (111.6, 64.6)
- moved C21 5.00 mm to (127.1, 91.3)
- moved Q8 5.00 mm to (126.7, 78.1)
- moved C11 5.00 mm to (120.0, 91.6)
- moved C2 5.00 mm to (100.5, 65.0)
- moved C22 5.00 mm to (139.3, 98.8)
- moved C23 5.00 mm to (139.3, 100.8)
- moved C24 5.00 mm to (147.0, 80.5)
- moved C25 5.00 mm to (146.9, 65.0)
- moved C3 5.00 mm to (96.0, 72.1)
- moved C31 5.00 mm to (108.4, 100.5)
- moved C33 5.00 mm to (132.0, 112.8)
- moved C34 5.00 mm to (135.5, 112.8)
- moved C4 5.00 mm to (99.3, 72.1)
- moved C5 5.00 mm to (102.6, 72.1)
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Connections:
- J2 pad 1: /GND -> GNDA
Routing:
- net VDD: track 49.9 -> 110.4 mm, vias 2 -> 6
- net VD: track 39.3 -> 93.8 mm, vias 2 -> 3
- net /CSPOUT: track 0.00 -> 38.2 mm, vias 17 -> 34
- net /MODE: track 4.34 -> 28.3 mm
- net /BOOST1: track 28.9 -> 15.4 mm
- net /SHDN: track 3.52 -> 15.7 mm, vias 0 -> 2
- net /GATEVCC: track 9.80 -> 20.6 mm, vias 0 -> 3
- net /EXTVCC: track 55.5 -> 45.6 mm
- net /SW2: track 55.4 -> 51.4 mm, vias 49 -> 48
- net /SW1: track 47.1 -> 49.9 mm, vias 49 -> 48
- net Net-(D3-Pad2): track 40.8 -> 43.4 mm
- net /BOOST2: track 20.6 -> 18.9 mm
- net /VC: track 33.2 -> 32.1 mm
- net Net-(Q3-Pad4): track 36.9 -> 37.9 mm
- net Net-(Q1-Pad4): track 41.0 -> 41.5 mm
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- added copper zone on F.Cu, net /GATEVCC
- added copper zone on B.Cu, net GNDA
- added copper zone on F.Cu, net GNDA
- added copper zone on In1.Cu, net GNDA
- added copper zone on In2.Cu, net GNDA
Other:
- board text added: "BURST"
- board text added: "DCM"
- board text added: "EXTVCC"
- board text added: "FCM"
- board text added: "IOUT"
- board text added: "VOUT"
