File: LT8705.sch (KiCad schematic (older format))
At the start: 64 parts, among them J1 XH-2, J2 HDR-M-2.54-1*4P, Q1 CSD19532Q5B, Q2 CSD19532Q5B, Q3 CSD19532Q5B, Q4 CSD19532Q5B, U1 LT8705EFE

Commit message: 1
Parts:
- removed R1, R5, R7: WSK06121L000FEA, _Acha:WSK06121L000FEA, symbol _Acha:WSK06121L000FEA
- added C10, C9: 4.7uF/100V, Capacitor_SMD:C_1210_3225Metric_Pad1.33x2.70mm_HandSolder, symbol LT8705-rescue:C-Device
- added D1, D2: ?, Diode_SMD:D_SMA-SMB_Universal_Handsoldering, symbol Device:D_Schottky
- added Q3, Q4, Q5, Q6: NC, Package_TO_SOT_SMD:TDSON-8-1, symbol LT8705-rescue:CSD19532Q5B-Transistor_FET
- added R1, R13, R8: WSK06125L000FEA, Resistor_SMD:R_Shunt_Vishay_WSKW0612, symbol Device:R_Shunt
- added R10, R4: 2R, Resistor_SMD:R_0603_1608Metric_Pad0.98x0.95mm_HandSolder, symbol LT8705-rescue:R-Device
- added R11, R3, R5, R9: 0, Resistor_SMD:R_0603_1608Metric_Pad0.98x0.95mm_HandSolder, symbol LT8705-rescue:R-Device
- added RV1: 50K, Potentiometer_THT:Potentiometer_Bourns_3296W_Vertical, symbol LT8705-rescue:R_POT-Device
- C1, C2: symbol Device:CP1 -> LT8705-rescue:CP1-Device
- C11: renamed from C5; symbol Device:C -> LT8705-rescue:C-Device
- C12: renamed from C7; symbol Device:C -> LT8705-rescue:C-Device
- C13: renamed from C9; symbol Device:C -> LT8705-rescue:C-Device
- C14: renamed from C11; symbol Device:C -> LT8705-rescue:C-Device
- C15: renamed from C13; symbol Device:C -> LT8705-rescue:C-Device
- C16: renamed from C14; symbol Device:C -> LT8705-rescue:C-Device
- C17: renamed from C15; symbol Device:CP1 -> LT8705-rescue:CP1-Device
- C18: renamed from C16; value C -> 100nF; symbol Device:C -> LT8705-rescue:C-Device
- C19: renamed from C17; symbol Device:C -> LT8705-rescue:C-Device
- C20: renamed from C18; symbol Device:C -> LT8705-rescue:C-Device
- C21: renamed from C19; symbol Device:CP1 -> LT8705-rescue:CP1-Device
- C22: renamed from C20; symbol Device:C -> LT8705-rescue:C-Device
- C23: renamed from C21; symbol Device:C -> LT8705-rescue:C-Device
- C24: renamed from C22; symbol Device:C -> LT8705-rescue:C-Device
- C25: renamed from C23; symbol Device:C -> LT8705-rescue:C-Device
- C26: renamed from C24; symbol Device:C -> LT8705-rescue:C-Device
- C27: renamed from C25; symbol Device:C -> LT8705-rescue:C-Device
- C28: renamed from C26; symbol Device:C -> LT8705-rescue:C-Device
- C29: renamed from C27; symbol Device:C -> LT8705-rescue:C-Device
- C3, C4: footprint Capacitor_SMD:C_1210_3225Metric_Pad1.42x2.65mm_HandSolder -> Capacitor_SMD:C_1210_3225Metric_Pad1.33x2.70mm_HandSolder; symbol Device:C -> LT8705-rescue:C-Device
- C30: renamed from C28; symbol Device:C -> LT8705-rescue:C-Device
- C31: renamed from C29; symbol Device:C -> LT8705-rescue:C-Device
- C32: renamed from C30; symbol Device:C -> LT8705-rescue:C-Device
- C33: renamed from C31; symbol Device:C -> LT8705-rescue:C-Device
- C34: renamed from C33; symbol Device:C -> LT8705-rescue:C-Device
- C35: renamed from C32; symbol Device:C -> LT8705-rescue:C-Device
- C5: renamed from C6; footprint Capacitor_SMD:C_1210_3225Metric_Pad1.42x2.65mm_HandSolder -> Capacitor_SMD:C_1210_3225Metric_Pad1.33x2.70mm_HandSolder; symbol Device:C -> LT8705-rescue:C-Device
- C6: renamed from C8; footprint Capacitor_SMD:C_1210_3225Metric_Pad1.42x2.65mm_HandSolder -> Capacitor_SMD:C_1210_3225Metric_Pad1.33x2.70mm_HandSolder; symbol Device:C -> LT8705-rescue:C-Device
- C7: renamed from C10; footprint Capacitor_SMD:C_1210_3225Metric_Pad1.42x2.65mm_HandSolder -> Capacitor_SMD:C_1210_3225Metric_Pad1.33x2.70mm_HandSolder; symbol Device:C -> LT8705-rescue:C-Device
- C8: renamed from C12; footprint Capacitor_SMD:C_1210_3225Metric_Pad1.42x2.65mm_HandSolder -> Capacitor_SMD:C_1210_3225Metric_Pad1.33x2.70mm_HandSolder; symbol Device:C -> LT8705-rescue:C-Device
- D3: renamed from D1; symbol Diode:1N4148W -> LT8705-rescue:1N4148W-Diode
- D4: renamed from D2; symbol Diode:1N4148W -> LT8705-rescue:1N4148W-Diode
- J1: symbol Connector_Generic:Conn_01x02 -> LT8705-rescue:Conn_01x02-Connector_Generic
- J2: symbol Connector_Generic:Conn_01x04 -> LT8705-rescue:Conn_01x04-Connector_Generic
- L1: symbol Device:L -> LT8705-rescue:L-Device
- Q1, Q2: symbol Transistor_FET:CSD19532Q5B -> LT8705-rescue:CSD19532Q5B-Transistor_FET
- Q7: renamed from Q3; symbol Transistor_FET:CSD19532Q5B -> LT8705-rescue:CSD19532Q5B-Transistor_FET
- Q8: renamed from Q4; symbol Transistor_FET:CSD19532Q5B -> LT8705-rescue:CSD19532Q5B-Transistor_FET
- R12: renamed from R6; footprint Resistor_SMD:R_0603_1608Metric_Pad1.05x0.95mm_HandSolder -> Resistor_SMD:R_0603_1608Metric_Pad0.98x0.95mm_HandSolder; symbol Device:R -> LT8705-rescue:R-Device
- R14: renamed from R8; footprint Resistor_SMD:R_0603_1608Metric_Pad1.05x0.95mm_HandSolder -> Resistor_SMD:R_0603_1608Metric_Pad0.98x0.95mm_HandSolder; symbol Device:R -> LT8705-rescue:R-Device
- R15: renamed from R9; footprint Resistor_SMD:R_0603_1608Metric_Pad1.05x0.95mm_HandSolder -> Resistor_SMD:R_0603_1608Metric_Pad0.98x0.95mm_HandSolder; symbol Device:R -> LT8705-rescue:R-Device
- R16: renamed from R10; footprint Resistor_SMD:R_0603_1608Metric_Pad1.05x0.95mm_HandSolder -> Resistor_SMD:R_0603_1608Metric_Pad0.98x0.95mm_HandSolder; symbol Device:R -> LT8705-rescue:R-Device
- R17: renamed from R11; footprint Resistor_SMD:R_0603_1608Metric_Pad1.05x0.95mm_HandSolder -> Resistor_SMD:R_0603_1608Metric_Pad0.98x0.95mm_HandSolder; symbol Device:R -> LT8705-rescue:R-Device
- R18: renamed from R12; footprint Resistor_SMD:R_0603_1608Metric_Pad1.05x0.95mm_HandSolder -> Resistor_SMD:R_0603_1608Metric_Pad0.98x0.95mm_HandSolder; symbol Device:R -> LT8705-rescue:R-Device
- R19: renamed from R13; footprint Resistor_SMD:R_0603_1608Metric_Pad1.05x0.95mm_HandSolder -> Resistor_SMD:R_0603_1608Metric_Pad0.98x0.95mm_HandSolder; symbol Device:R -> LT8705-rescue:R-Device
- R2: footprint Resistor_SMD:R_0603_1608Metric_Pad1.05x0.95mm_HandSolder -> Resistor_SMD:R_0603_1608Metric_Pad0.98x0.95mm_HandSolder; symbol Device:R -> LT8705-rescue:R-Device
- R20: renamed from R14; footprint Resistor_SMD:R_0603_1608Metric_Pad1.05x0.95mm_HandSolder -> Resistor_SMD:R_0603_1608Metric_Pad0.98x0.95mm_HandSolder; symbol Device:R -> LT8705-rescue:R-Device
- R21: renamed from R15; value 40.2K -> NC; footprint Resistor_SMD:R_0603_1608Metric_Pad1.05x0.95mm_HandSolder -> Resistor_SMD:R_0603_1608Metric_Pad0.98x0.95mm_HandSolder; symbol Device:R -> LT8705-rescue:R-Device
- R22: renamed from R16; footprint Resistor_SMD:R_0603_1608Metric_Pad1.05x0.95mm_HandSolder -> Resistor_SMD:R_0603_1608Metric_Pad0.98x0.95mm_HandSolder; symbol Device:R -> LT8705-rescue:R-Device
- R23: renamed from R17; footprint Resistor_SMD:R_0603_1608Metric_Pad1.05x0.95mm_HandSolder -> Resistor_SMD:R_0603_1608Metric_Pad0.98x0.95mm_HandSolder; symbol Device:R -> LT8705-rescue:R-Device
- R24: renamed from R18; footprint Resistor_SMD:R_0603_1608Metric_Pad1.05x0.95mm_HandSolder -> Resistor_SMD:R_0603_1608Metric_Pad0.98x0.95mm_HandSolder; symbol Device:R -> LT8705-rescue:R-Device
- R25: renamed from R19; footprint Resistor_SMD:R_0603_1608Metric_Pad1.05x0.95mm_HandSolder -> Resistor_SMD:R_0603_1608Metric_Pad0.98x0.95mm_HandSolder; symbol Device:R -> LT8705-rescue:R-Device
- R6: renamed from R3; footprint Resistor_SMD:R_0603_1608Metric_Pad1.05x0.95mm_HandSolder -> Resistor_SMD:R_0603_1608Metric_Pad0.98x0.95mm_HandSolder; symbol Device:R -> LT8705-rescue:R-Device
- R7: renamed from R4; footprint Resistor_SMD:R_0603_1608Metric_Pad1.05x0.95mm_HandSolder -> Resistor_SMD:R_0603_1608Metric_Pad0.98x0.95mm_HandSolder; symbol Device:R -> LT8705-rescue:R-Device
- RV2: renamed from RV1; symbol Device:R_POT -> LT8705-rescue:R_POT-Device
- RV3: renamed from RV2; symbol Device:R_POT -> LT8705-rescue:R_POT-Device
- U1: symbol _Acha:LT8705EFE -> LT8705-rescue:LT8705EFE-_Acha
Connections:
- wire segments 158 -> 184
- no-connect marks 0 -> 2
Other:
- moved on the sheet: R2, R21, R6, R7

Commit message: Updated
Parts:
- removed R1, R13: WSK06125L000FEA, Resistor_SMD:R_Shunt_Vishay_WSKW0612, symbol Device:R_Shunt
- added R1, R13: R, symbol Device:R
Connections:
- wire segments 184 -> 188
Other:
- moved on the sheet: C10, C7, C8, C9
Changed lines of the file:
@@
-$EndComp
-$Comp
-L LT8705-rescue:CP1-Device C1
-U 1 1 6115514A
-P 975 1000
-F 0 "C1" H 925 750 50  0000 L CNN
-F 1 "220uF/100V" H 875 650 50  0000 L CNN
-F 2 "Capacitor_THT:C_Radial_D12.5mm_H25.0mm_P5.00mm" H 975 1000 50  0001 C CNN
-F 3 "~" H 975 1000 50  0001 C CNN
-	1    975  1000
-	1    0    0    -1
 $EndComp
 $Comp
@@
 	9900 3800 10250 3800
 Wire Wire Line
-	825  850  975  850
-Wire Wire Line
 	3350 1900 3125 1900
 Text Label 3125 1900 0    50   ~ 0
@@
 	1    0    0    -1
 $EndComp
-Wire Wire Line
-	2825 700  3075 700
-Wire Wire Line
-	3275 700  3575 700
-Text Label 2825 700  0    50   ~ 0
-CSPIN
-Text Label 3300 700  0    50   ~ 0
-CSNIN
 Connection ~ 6875 900
 Wire Wire Line
-	6425 750  6725 750
-Wire Wire Line
-	6225 750  5925 750
-Text Label 5925 750  0    50   ~ 0
+	6475 750  6775 750
+Wire Wire Line
+	6175 750  5875 750
+Text Label 5875 750  0    50   ~ 0
 CSPOUT
-Text Label 6450 750  0    50   ~ 0
+Text Label 6500 750  0    50   ~ 0
 CSNOUT
-Wire Wire Line
-	2900 1150 2700 1150
-Connection ~ 975  1150
 Connection ~ 1200 1150
-Wire Wire Line
-	1200 1150 975  1150
 Connection ~ 1500 1150
 Wire Wire Line
@@
 	1    0    0    -1
 $EndComp
-Wire Wire Line
-	675  1150 975  1150
 Wire Wire Line
 	8400 1200 8600 1200
@@
 Connection ~ 1700 850
 Connection ~ 1900 850
-Connection ~ 2100 850
 Wire Wire Line
 	1500 850  1700 850
@@
 Wire Wire Line
 	1900 850  2100 850
-Wire Wire Line
-	2100 850  2300 850
-Connection ~ 975  850
-Wire Wire Line
-	975  850  1200 850
 $Comp
 L LT8705-rescue:C-Device C7
 U 1 1 611536ED
-P 2300 1000
-F 0 "C7" H 2250 750 50  0000 L CNN
-F 1 "4.7uF/100V" H 2250 675 50  0001 L CNN
-F 2 "Capacitor_SMD:C_1210_3225Metric_Pad1.33x2.70mm_HandSolder" H 2338 850 50  0001 C CNN
-F 3 "~" H 2300 1000 50  0001 C CNN
-	1    2300 1000
-	1    0    0    -1
-$EndComp
-Connection ~ 2300 850
-Wire Wire Line
-	2300 850  2500 850
+P 2600 1000
+F 0 "C7" H 2550 750 50  0000 L CNN
+F 1 "4.7uF/100V" H 2550 675 50  0001 L CNN
+F 2 "Capacitor_SMD:C_1210_3225Metric_Pad1.33x2.70mm_HandSolder" H 2638 850 50  0001 C CNN
+F 3 "~" H 2600 1000 50  0001 C CNN
+	1    2600 1000
+	1    0    0    -1
+$EndComp
 $Comp
 L LT8705-rescue:C-Device C8
 U 1 1 61153F53
-P 2500 1000
-F 0 "C8" H 2450 750 50  0000 L CNN
-F 1 "4.7uF/100V" H 2450 675 50  0001 L CNN
-F 2 "Capacitor_SMD:C_1210_3225Metric_Pad1.33x2.70mm_HandSolder" H 2538 850 50  0001 C CNN
-F 3 "~" H 2500 1000 50  0001 C CNN
-	1    2500 1000
+P 2800 1000
+F 0 "C8" H 2750 750 50  0000 L CNN
+F 1 "4.7uF/100V" H 2750 675 50  0001 L CNN
+F 2 "Capacitor_SMD:C_1210_3225Metric_Pad1.33x2.70mm_HandSolder" H 2838 850 50  0001 C CNN
+F 3 "~" H 2800 1000 50  0001 C CNN
+	1    2800 1000
 	1    0    0    -1
 $EndComp
@@
 Wire Wire Line
 	2100 1150 1900 1150
-Connection ~ 2300 1150
-Wire Wire Line
-	2300 1150 2100 1150
 $Comp
 L LT8705-rescue:C-Device C28
@@
 	3850 2475 3750 2475
 Connection ~ 3750 2475
-$Comp
-L Device:R_Shunt R1
-U 1 1 6116C974
-P 3175 850
-F 0 "R1" V 3500 850 50  0000 C CNN
-F 1 "WSK06125L000FEA" V 3425 825 50  0000 C CNN
-F 2 "Resistor_SMD:R_Shunt_Vishay_WSKW0612" V 3105 850 50  0001 C CNN
-F 3 "~" H 3175 850 50  0001 C CNN
-	1    3175 850
-	0    -1   -1   0
-$EndComp
-Wire Wire Line
-	3375 850  3650 850
-$Comp
-L Device:R_Shunt R13
-U 1 1 611A11FE
-P 6325 900
-F 0 "R13" V 6650 900 50  0000 C CNN
-F 1 "WSK06125L000FEA" V 6575 875 50  0000 C CNN
-F 2 "Resistor_SMD:R_Shunt_Vishay_WSKW0612" V 6255 900 50  0001 C CNN
-F 3 "~" H 6325 900 50  0001 C CNN
-	1    6325 900
-	0    -1   -1   0
-$EndComp
 Wire Wire Line
 	5750 900  6075 900
-Wire Wire Line
-	6525 900  6875 900
 $Comp
 L LT8705-rescue:R-Device R3
@@
 	6075 1400 6075 900
 Connection ~ 6075 900
-Wire Wire Line
-	6075 900  6125 900
 $Comp
 L LT8705-rescue:C-Device C9
 U 1 1 6146E0DE
-P 2700 1000
-F 0 "C9" H 2650 750 50  0000 L CNN
-F 1 "4.7uF/100V" H 2650 675 50  0001 L CNN
-F 2 "Capacitor_SMD:C_1210_3225Metric_Pad1.33x2.70mm_HandSolder" H 2738 850 50  0001 C CNN
-F 3 "~" H 2700 1000 50  0001 C CNN
-	1    2700 1000
+P 3000 1000
+F 0 "C9" H 2950 750 50  0000 L CNN
+F 1 "4.7uF/100V" H 2950 675 50  0001 L CNN
+F 2 "Capacitor_SMD:C_1210_3225Metric_Pad1.33x2.70mm_HandSolder" H 3038 850 50  0001 C CNN
+F 3 "~" H 3000 1000 50  0001 C CNN
+	1    3000 1000
 	1    0    0    -1
 $EndComp
@@
 L LT8705-rescue:C-Device C10
 U 1 1 6146E505
-P 2900 1000
-F 0 "C10" H 2850 750 50  0000 L CNN
-F 1 "4.7uF/100V" H 2850 675 50  0001 L CNN
-F 2 "Capacitor_SMD:C_1210_3225Metric_Pad1.33x2.70mm_HandSolder" H 2938 850 50  0001 C CNN
-F 3 "~" H 2900 1000 50  0001 C CNN
-	1    2900 1000
-	1    0    0    -1
-$EndComp
-Connection ~ 2500 1150
-Wire Wire Line
-	2500 1150 2300 1150
-Connection ~ 2700 1150
-Wire Wire Line
-	2700 1150 2500 1150
-Wire Wire Line
-	2500 850  2700 850
-Connection ~ 2500 850
-Connection ~ 2700 850
-Wire Wire Line
-	2700 850  2900 850
-Connection ~ 2900 850
-Wire Wire Line
-	2900 850  2975 850
+P 3200 1000
+F 0 "C10" H 3150 750 50  0000 L CNN
+F 1 "4.7uF/100V" H 3150 675 50  0001 L CNN
+F 2 "Capacitor_SMD:C_1210_3225Metric_Pad1.33x2.70mm_HandSolder" H 3238 850 50  0001 C CNN
+F 3 "~" H 3200 1000 50  0001 C CNN
+	1    3200 1000
+	1    0    0    -1
+$EndComp
 $Comp
 L LT8705-rescue:R_POT-Device RV1
@@
 Wire Wire Line
 	5750 1400 5775 1400
+Wire Wire Line
+	2100 1150 2600 1150
+Connection ~ 2600 1150
+Wire Wire Line
+	2600 1150 2800 1150
+Connection ~ 2800 1150
+Wire Wire Line
+	2800 1150 3000 1150
+Connection ~ 3000 1150
+Wire Wire Line
+	3000 1150 3200 1150
+Connection ~ 2100 850
+Connection ~ 2600 850
+Wire Wire Line
+	2600 850  2800 850
+Connection ~ 2800 850
+Wire Wire Line
+	2800 850  3000 850
+Connection ~ 3000 850
+Wire Wire Line
+	3000 850  3200 850
+Connection ~ 3200 850
+Wire Wire Line
+	3200 850  3650 850
+Wire Wire Line
+	675  1150 975  1150
+Wire Wire Line
+	1200 1150 975  1150
+Connection ~ 975  1150
+Wire Wire Line
+	975  850  1200 850
+Wire Wire Line
+	825  850  975  850
+Connection ~ 975  850
+$Comp
+L LT8705-rescue:CP1-Device C1
+U 1 1 6115514A
+P 975 1000
+F 0 "C1" H 925 750 50  0000 L CNN
+F 1 "220uF/100V" H 875 650 50  0000 L CNN
+F 2 "Capacitor_THT:C_Radial_D12.5mm_H25.0mm_P5.00mm" H 975 1000 50  0001 C CNN
+F 3 "~" H 975 1000 50  0001 C CNN
+	1    975  1000
+	1    0    0    -1
+$EndComp
+Text Label 2525 700  0    50   ~ 0
+CSNIN
+Text Label 1950 700  0    50   ~ 0
+CSPIN
+Wire Wire Line
+	2500 700  2800 700
+Wire Wire Line
+	1950 700  2200 700
+$Comp
+L Device:R R1
+U 1 1 6121B64F
+P 2350 850
+F 0 "R1" V 2143 850 50  0000 C CNN
+F 1 "R" V 2234 850 50  0000 C CNN
+F 2 "" V 2280 850 50  0001 C CNN
+F 3 "~" H 2350 850 50  0001 C CNN
+	1    2350 850
+	0    1    1    0
+$EndComp
+Wire Wire Line
+	2100 850  2200 850
+Wire Wire Line
+	2200 700  2200 850
+Connection ~ 2200 850
+Wire Wire Line
+	2500 850  2600 850
+Wire Wire Line
+	2500 700  2500 850
+Connection ~ 2500 850
+$Comp
+L Device:R R13
+U 1 1 61271573
+P 6325 900
+F 0 "R13" V 6118 900 50  0000 C CNN
+F 1 "R" V 6209 900 50  0000 C CNN
+F 2 "" V 6255 900 50  0001 C CNN
+F 3 "~" H 6325 900 50  0001 C CNN
+	1    6325 900
+	0    1    1    0
+$EndComp
+Wire Wire Line
+	6075 900  6175 900
+Wire Wire Line
+	6175 750  6175 900
+Connection ~ 6175 900
+Wire Wire Line
+	6475 900  6875 900
+Wire Wire Line
+	6475 750  6475 900
+Connection ~ 6475 900
 $EndSCHEMATC

Commit message: updated
Parts:
- removed R8: WSK06125L000FEA, Resistor_SMD:R_Shunt_Vishay_WSKW0612, symbol Device:R_Shunt
- added R26: 0, Resistor_SMD:R_0603_1608Metric_Pad0.98x0.95mm_HandSolder, symbol LT8705-rescue:R-Device
- added R8: R005, _Acha:R_1225_3263Metric, symbol Device:R
- R1: value R -> 0R; footprint (none) -> _Acha:R_0612_1632Metric
- R13: value R -> R005; footprint (none) -> _Acha:R_0612_1632Metric
- renumbered C9 to C10, C12 to C11, C10 to C12, C22 to C17, C23 to C18, C24 to C19, C25 to C20, C18 to C21, C19 to C22, C20 to C23, C17 to C24, C21 to C25, C11 to C9
Connections:
- wire segments 188 -> 191
Other:
- moved on the sheet: C16, C17, C18, C19, C20, C24, C25, R13, R7

Commit message: 1
Parts:
- added R22: R, Resistor_SMD:R_0603_1608Metric_Pad0.98x0.95mm_HandSolder, symbol Device:R
- renumbered R26 to R1, R9 to R10, R10 to R11, R11 to R12, R12 to R13, R13 to R14, R14 to R15, R15 to R16, R16 to R17, R17 to R18, R18 to R19, R1 to R2, R19 to R20, R20 to R21, R21 to R23, R22 to R24, R23 to R25, R24 to R26, R25 to R27, R2 to R3, R3 to R4, R4 to R5, R5 to R6, R6 to R7, R7 to R8, R8 to R9
Connections:
- wire segments 191 -> 195
Changed lines of the file:
@@
 	9500 475  9500 6525
 $Comp
-L LT8705-rescue:R-Device R17
+L LT8705-rescue:R-Device R18
 U 1 1 6110C445
 P 9900 875
-F 0 "R17" H 9970 921 50  0000 L CNN
+F 0 "R18" H 9970 921 50  0000 L CNN
 F 1 "71.5K" H 9970 830 50  0000 L CNN
 F 2 "Resistor_SMD:R_0603_1608Metric_Pad0.98x0.95mm_HandSolder" V 9830 875 50  0001 C CNN
@@
 $EndComp
 $Comp
-L LT8705-rescue:R-Device R18
+L LT8705-rescue:R-Device R19
 U 1 1 6110D65E
 P 9900 1175
-F 0 "R18" H 9970 1221 50  0000 L CNN
+F 0 "R19" H 9970 1221 50  0000 L CNN
 F 1 "20K" H 9970 1130 50  0000 L CNN
 F 2 "Resistor_SMD:R_0603_1608Metric_Pad0.98x0.95mm_HandSolder" V 9830 1175 50  0001 C CNN
@@
 $EndComp
 $Comp
-L LT8705-rescue:R-Device R24
+L LT8705-rescue:R-Device R26
 U 1 1 61120C98
 P 10825 925
-F 0 "R24" H 10895 971 50  0000 L CNN
+F 0 "R26" H 10895 971 50  0000 L CNN
 F 1 "NC" H 10895 880 50  0000 L CNN
 F 2 "Resistor_SMD:R_0603_1608Metric_Pad0.98x0.95mm_HandSolder" V 10755 925 50  0001 C CNN
@@
 $EndComp
 $Comp
-L LT8705-rescue:R-Device R25
+L LT8705-rescue:R-Device R27
 U 1 1 6112176C
 P 10825 1225
-F 0 "R25" H 10895 1271 50  0000 L CNN
+F 0 "R27" H 10895 1271 50  0000 L CNN
 F 1 "NC" H 10895 1180 50  0000 L CNN
 F 2 "Resistor_SMD:R_0603_1608Metric_Pad0.98x0.95mm_HandSolder" V 10755 1225 50  0001 C CNN
@@
 FBOUT
 $Comp
-L LT8705-rescue:R-Device R15
+L LT8705-rescue:R-Device R16
 U 1 1 611334BB
 P 9675 2025
-F 0 "R15" H 9745 2071 50  0000 L CNN
+F 0 "R16" H 9745 2071 50  0000 L CNN
 F 1 "NC" H 9745 1980 50  0000 L CNN
 F 2 "Resistor_SMD:R_0603_1608Metric_Pad0.98x0.95mm_HandSolder" V 9605 2025 50  0001 C CNN
@@
 $EndComp
 $Comp
-L LT8705-rescue:R-Device R16
+L LT8705-rescue:R-Device R17
 U 1 1 6113415C
 P 9675 2325
-F 0 "R16" H 9745 2371 50  0000 L CNN
+F 0 "R17" H 9745 2371 50  0000 L CNN
 F 1 "NC" H 9745 2280 50  0000 L CNN
 F 2 "Resistor_SMD:R_0603_1608Metric_Pad0.98x0.95mm_HandSolder" V 9605 2325 50  0001 C CNN
@@
 $EndComp
 $Comp
-L LT8705-rescue:R-Device R20
+L LT8705-rescue:R-Device R21
 U 1 1 611349B0
 P 9950 2025
-F 0 "R20" H 10020 2071 50  0000 L CNN
+F 0 "R21" H 10020 2071 50  0000 L CNN
 F 1 "0R" H 10020 1980 50  0000 L CNN
 F 2 "Resistor_SMD:R_0603_1608Metric_Pad0.98x0.95mm_HandSolder" V 9880 2025 50  0001 C CNN
@@
 	9500 2825 11225 2825
 $Comp
-L LT8705-rescue:R-Device R22
+L LT8705-rescue:R-Device R24
 U 1 1 6113FA46
 P 10775 2175
-F 0 "R22" H 10845 2221 50  0000 L CNN
+F 0 "R24" H 10845 2221 50  0000 L CNN
 F 1 "110K" H 10845 2130 50  0000 L CNN
 F 2 "Resistor_SMD:R_0603_1608Metric_Pad0.98x0.95mm_HandSolder" V 10705 2175 50  0001 C CNN
@@
 $EndComp
 $Comp
-L LT8705-rescue:R-Device R14
+L LT8705-rescue:R-Device R15
 U 1 1 61143E4D
 P 9650 3250
-F 0 "R14" H 9720 3296 50  0000 L CNN
+F 0 "R15" H 9720 3296 50  0000 L CNN
 F 1 "0R" H 9720 3205 50  0000 L CNN
 F 2 "Resistor_SMD:R_0603_1608Metric_Pad0.98x0.95mm_HandSolder" V 9580 3250 50  0001 C CNN
@@
 IMON_IN
 $Comp
-L LT8705-rescue:R-Device R21
+L LT8705-rescue:R-Device R23
 U 1 1 61154E98
 P 10700 3250
-F 0 "R21" H 10750 3250 50  0000 L CNN
+F 0 "R23" H 10750 3250 50  0000 L CNN
 F 1 "NC" H 10750 3175 50  0000 L CNN
 F 2 "Resistor_SMD:R_0603_1608Metric_Pad0.98x0.95mm_HandSolder" V 10630 3250 50  0001 C CNN
@@
 $EndComp
 $Comp
-L LT8705-rescue:R-Device R19
+L LT8705-rescue:R-Device R20
 U 1 1 610F6B79
 P 9900 3975
-F 0 "R19" H 9970 4021 50  0000 L CNN
+F 0 "R20" H 9970 4021 50  0000 L CNN
 F 1 "4R" H 9970 3930 50  0000 L CNN
 F 2 "Resistor_SMD:R_0603_1608Metric_Pad0.98x0.95mm_HandSolder" V 9830 3975 50  0001 C CNN
@@
 $EndComp
 $Comp
-L LT8705-rescue:R-Device R23
+L LT8705-rescue:R-Device R25
 U 1 1 61109B1E
 P 10775 4250
-F 0 "R23" V 10625 4250 50  0000 C CNN
+F 0 "R25" V 10625 4250 50  0000 C CNN
 F 1 "NC" V 10700 4250 50  0000 C CNN
 F 2 "Resistor_SMD:R_0603_1608Metric_Pad0.98x0.95mm_HandSolder" V 10705 4250 50  0001 C CNN
@@
 BG1
 $Comp
-L LT8705-rescue:R-Device R2
+L LT8705-rescue:R-Device R3
 U 1 1 6113BEEA
 P 3350 1200
-F 0 "R2" H 3420 1246 50  0000 L CNN
+F 0 "R3" H 3420 1246 50  0000 L CNN
 F 1 "2R" H 3420 1155 50  0000 L CNN
 F 2 "Resistor_SMD:R_0603_1608Metric_Pad0.98x0.95mm_HandSolder" V 3280 1200 50  0001 C CNN
@@
 TG2
 $Comp
-L LT8705-rescue:R-Device R12
+L LT8705-rescue:R-Device R13
 U 1 1 61145A8C
 P 5450 1750
-F 0 "R12" H 5520 1796 50  0000 L CNN
+F 0 "R13" H 5520 1796 50  0000 L CNN
 F 1 "2R" H 5520 1705 50  0000 L CNN
 F 2 "Resistor_SMD:R_0603_1608Metric_Pad0.98x0.95mm_HandSolder" V 5380 1750 50  0001 C CNN
@@
 $EndComp
 $Comp
-L LT8705-rescue:R-Device R6
+L LT8705-rescue:R-Device R7
 U 1 1 611B36C2
 P 4500 2275
-F 0 "R6" V 4575 2175 50  0000 C CNN
+F 0 "R7" V 4575 2175 50  0000 C CNN
 F 1 "10R" V 4575 2325 50  0000 C CNN
 F 2 "Resistor_SMD:R_0603_1608Metric_Pad0.98x0.95mm_HandSolder" V 4430 2275 50  0001 C CNN
@@
 $EndComp
 $Comp
-L LT8705-rescue:R-Device R7
+L LT8705-rescue:R-Device R8
 U 1 1 611B48A9
 P 4500 2550
-F 0 "R7" V 4600 2450 50  0000 C CNN
+F 0 "R8" V 4600 2450 50  0000 C CNN
 F 1 "10R" V 4600 2600 50  0000 C CNN
 F 2 "Resistor_SMD:R_0603_1608Metric_Pad0.98x0.95mm_HandSolder" V 4430 2550 50  0001 C CNN
@@
 	5750 900  6075 900
 $Comp
-L LT8705-rescue:R-Device R3
+L LT8705-rescue:R-Device R4
 U 1 1 611F9CD2
 P 3350 1750
-F 0 "R3" H 3420 1796 50  0000 L CNN
+F 0 "R4" H 3420 1796 50  0000 L CNN
 F 1 "0" H 3420 1705 50  0000 L CNN
 F 2 "Resistor_SMD:R_0603_1608Metric_Pad0.98x0.95mm_HandSolder" V 3280 1750 50  0001 C CNN
@@
 $EndComp
 $Comp
-L LT8705-rescue:R-Device R11
+L LT8705-rescue:R-Device R12
 U 1 1 6120565D
 P 5450 950
-F 0 "R11" H 5520 996 50  0000 L CNN
+F 0 "R12" H 5520 996 50  0000 L CNN
 F 1 "0" H 5520 905 50  0000 L CNN
 F 2 "Resistor_SMD:R_0603_1608Metric_Pad0.98x0.95mm_HandSolder" V 5380 950 50  0001 C CNN
@@
 	4225 850  3650 850
 $Comp
-L LT8705-rescue:R-Device R4
+L LT8705-rescue:R-Device R5
 U 1 1 612B25CA
 P 3925 1200
-F 0 "R4" H 3995 1246 50  0000 L CNN
+F 0 "R5" H 3995 1246 50  0000 L CNN
 F 1 "2R" H 3995 1155 50  0000 L CNN
 F 2 "Resistor_SMD:R_0603_1608Metric_Pad0.98x0.95mm_HandSolder" V 3855 1200 50  0001 C CNN
@@
 BG1
 $Comp
-L LT8705-rescue:R-Device R5
+L LT8705-rescue:R-Device R6
 U 1 1 612DD823
 P 3925 1750
-F 0 "R5" H 3995 1796 50  0000 L CNN
+F 0 "R6" H 3995 1796 50  0000 L CNN
 F 1 "0" H 3995 1705 50  0000 L CNN
 F 2 "Resistor_SMD:R_0603_1608Metric_Pad0.98x0.95mm_HandSolder" V 3855 1750 50  0001 C CNN
@@
 TG2
 $Comp
-L LT8705-rescue:R-Device R9
+L LT8705-rescue:R-Device R10
 U 1 1 6133D0FB
 P 4975 950
-F 0 "R9" H 5045 996 50  0000 L CNN
+F 0 "R10" H 5045 996 50  0000 L CNN
 F 1 "0" H 5045 905 50  0000 L CNN
 F 2 "Resistor_SMD:R_0603_1608Metric_Pad0.98x0.95mm_HandSolder" V 4905 950 50  0001 C CNN
@@
 	5450 1900 5675 1900
 $Comp
-L LT8705-rescue:R-Device R10
+L LT8705-rescue:R-Device R11
 U 1 1 61366F42
 P 4975 1750
-F 0 "R10" H 5045 1796 50  0000 L CNN
+F 0 "R11" H 5045 1796 50  0000 L CNN
 F 1 "2R" H 5045 1705 50  0000 L CNN
 F 2 "Resistor_SMD:R_0603_1608Metric_Pad0.98x0.95mm_HandSolder" V 4905 1750 50  0001 C CNN
@@
 	1950 700  2200 700
 $Comp
-L Device:R R1
+L Device:R R2
 U 1 1 6121B64F
 P 2350 850
-F 0 "R1" V 2143 850 50  0000 C CNN
+F 0 "R2" V 2143 850 50  0000 C CNN
 F 1 "0R" V 2234 850 50  0000 C CNN
 F 2 "_Acha:R_0612_1632Metric" V 2280 850 50  0001 C CNN
@@
 Connection ~ 2500 850
 $Comp
-L Device:R R13
+L Device:R R14
 U 1 1 61271573
 P 7400 900
-F 0 "R13" V 7193 900 50  0000 C CNN
+F 0 "R14" V 7193 900 50  0000 C CNN
 F 1 "R005" V 7284 900 50  0000 C CNN
 F 2 "_Acha:R_0612_1632Metric" V 7330 900 50  0001 C CNN
@@
 	4475 2175 4800 2175
 $Comp
-L Device:R R8
+L Device:R R9
 U 1 1 61226C1E
 P 4800 2425
-F 0 "R8" V 4593 2425 50  0000 C CNN
+F 0 "R9" V 4593 2425 50  0000 C CNN
 F 1 "R005" V 4684 2425 50  0000 C CNN
 F 2 "_Acha:R_1225_3263Metric" V 4730 2425 50  0001 C CNN
@@
 	3750 2275 3750 2550
 $Comp
-L LT8705-rescue:R-Device R26
+L LT8705-rescue:R-Device R1
 U 1 1 613A0A49
 P 2075 2650
-F 0 "R26" H 2145 2696 50  0000 L CNN
+F 0 "R1" H 2145 2696 50  0000 L CNN
 F 1 "0" H 2145 2605 50  0000 L CNN
 F 2 "Resistor_SMD:R_0603_1608Metric_Pad0.98x0.95mm_HandSolder" V 2005 2650 50  0001 C CNN
@@
 Wire Wire Line
 	4650 2550 4800 2550
+Wire Wire Line
+	10000 5150 10100 5150
+Wire Wire Line
+	10100 5150 10100 5450
+Connection ~ 10000 5150
+$Comp
+L Device:R R22
+U 1 1 61231BF9
+P 10100 5600
+F 0 "R22" H 10170 5646 50  0000 L CNN
+F 1 "R" H 10170 5555 50  0000 L CNN
+F 2 "Resistor_SMD:R_0603_1608Metric_Pad0.98x0.95mm_HandSolder" V 10030 5600 50  0001 C CNN
+F 3 "~" H 10100 5600 50  0001 C CNN
+	1    10100 5600
+	1    0    0    -1
+$EndComp
+Wire Wire Line
+	10100 5750 10100 5800
+Wire Wire Line
+	10100 5800 9725 5800
+Text Label 9725 5800 0    50   ~ 0
+VOUT
+Text Label 8800 900  0    50   ~ 0
+VOUT
 $EndSCHEMATC

Commit message: 1
Connections:
- net labels removed: GND
Changed lines of the file:
@@
 MODE
 Text Label 10700 5450 0    50   ~ 0
-GND
+GNDA
 $Comp
 L LT8705-rescue:GNDA-power #PWR03
